File: eagle/808_noise.brd (EAGLE design)
At the start: 100.6 x 80 mm, 25 parts, among them IC1 TL072P, Q1 2N3904

Commit message: with mods
Parts:
- removed R127: 47K, TR808clone:0207/7
- added C1: 10uF, rcl:B45181A
- R129: value 330K -> 0R
- R131: value 300K -> 100K
- moved C32 7.24 mm to (28.6, 22.2)
- moved R132 2.84 mm to (20.3, 22.9), turned to 180 degrees
- moved R133 2.84 mm to (20.3, 20.3), turned to 0 degrees
- moved C33 1.42 mm to (9.53, 24.1)
Connections:
- removed net N$228: R127.2, TM4.A
- new net N$1: C1.+, TM4.A
- net GND: now also C1.-; no longer R127.1
Routing:
- net GND: track 162.8 -> 170.1 mm
- net N$228: track 6.22 -> 0.00 mm
- net N$1: track 0.00 -> 6.13 mm
- net N$493: track 8.23 -> 4.55 mm
- net N$494: track 15.2 -> 16.6 mm
- net WN: track 102.7 -> 103.9 mm
