File: eagle/808_noise.sch (EAGLE design)
At the start: 20 parts, among them IC1 TL072P, Q1 2N3904, U24 µPC4558C

Commit message: routed
Parts:
- removed U24: µPC4558C, TR808clone:µPC4558C
- added C5, C7: 10u, rcl:CPOL-USB45181A
- added C8, C9: 100n, rcl:C-US050-024X044
- added U$2, U$3: FB, adafruit:FB
Connections:
- new net N$11: U$1.+12V, U$2.1
- new net N$18: U$1.-12V, U$3.1
- net +15V: now also C5.+, C8.1, IC1P.V+, U$2.2; no longer U$1.+12V, U24G$3.V+
- net -15V: now also C7.-, C9.2, IC1P.V-, U$3.2; no longer U$1.-12V, U24G$3.V-
- net GND: now also C5.-, C7.+, C8.2, C9.1
Other:
- moved on the sheet: U$1

Commit message: with mods
Parts:
- removed R127: 47K, TR808clone:R-EU_0207/7
- added C1: 10uF, rcl:CPOL-USB45181A
- R129: value 330K -> 0R
- R131: value 300K -> 100K
Connections:
- removed net N$228: R127.2, TM4.A
- new net N$1: C1.+, TM4.A
- net GND: now also C1.-; no longer R127.1
Other:
- moved on the sheet: R129
Changed lines of the file:
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@@
 <?xml version="1.0" encoding="utf-8"?>
 <!DOCTYPE eagle SYSTEM "eagle.dtd">
-<eagle version="7.2.0">
+<eagle version="7.1.0">
 <drawing>
 <settings>
@@
 <part name="R130" library="TR808clone" deviceset="R-EU_" device="0207/7" value="1M"/>
 <part name="R132" library="TR808clone" deviceset="R-EU_" device="0207/7" value="22K"/>
-<part name="R131" library="TR808clone" deviceset="R-EU_" device="0207/7" value="300K"/>
+<part name="R131" library="TR808clone" deviceset="R-EU_" device="0207/7" value="100K"/>
 <part name="V303" library="supply1" deviceset="GND" device=""/>
 <part name="V304" library="supply1" deviceset="GND" device=""/>
-<part name="R127" library="TR808clone" deviceset="R-EU_" device="0207/7" value="47K"/>
 <part name="V305" library="supply1" deviceset="GND" device=""/>
 <part name="C29" library="TR808clone" deviceset="CPOL-EU" device="E2.5-5" value="47/16"/>
@@
 <part name="R124" library="TR808clone" deviceset="R-EU_" device="0207/7" value="100R"/>
 <part name="C31" library="TR808clone" deviceset="CPOL-EU" device="E2.5-5" value="1/50"/>
-<part name="R129" library="TR808clone" deviceset="R-EU_" device="0207/7" value="330K"/>
 <part name="R128" library="TR808clone" deviceset="R-EU_" device="0207/7" value="1M"/>
 <part name="C32" library="TR808clone" deviceset="C-EU" device="050-024X044" value="39n"/>
@@
 <part name="C8" library="rcl" deviceset="C-US" device="050-024X044" value="100n"/>
 <part name="C9" library="rcl" deviceset="C-US" device="050-024X044" value="100n"/>
+<part name="C1" library="rcl" deviceset="CPOL-US" device="B45181A" value="10uF"/>
+<part name="R129" library="TR808clone" deviceset="R-EU_" device="0207/7" value="0R"/>
 </parts>
 <sheets>
@@
 <instance part="V303" gate="1" x="20.32" y="2.54"/>
 <instance part="V304" gate="1" x="38.1" y="2.54"/>
-<instance part="R127" gate="G$1" x="27.94" y="43.18" smashed="yes">
-<attribute name="NAME" x="24.13" y="44.6786" size="1.778" layer="95"/>
-<attribute name="VALUE" x="24.13" y="39.878" size="1.778" layer="96"/>
-</instance>
-<instance part="V305" gate="1" x="22.86" y="38.1"/>
+<instance part="V305" gate="1" x="22.86" y="35.56"/>
 <instance part="C29" gate="G$1" x="5.08" y="17.78"/>
 <instance part="V306" gate="1" x="5.08" y="2.54"/>
 <instance part="R124" gate="G$1" x="5.08" y="33.02" rot="R90"/>
 <instance part="C31" gate="G$1" x="30.48" y="22.86" rot="R90"/>
-<instance part="R129" gate="G$1" x="38.1" y="38.1" rot="R270"/>
 <instance part="R128" gate="G$1" x="10.16" y="27.94" rot="R180"/>
 <instance part="C32" gate="G$1" x="73.66" y="27.94" rot="R90"/>
@@
 <instance part="C9" gate="G$1" x="40.64" y="73.66"/>
 <instance part="IC1" gate="P" x="15.24" y="50.8"/>
+<instance part="C1" gate="G$1" x="27.94" y="43.18" rot="R270"/>
+<instance part="R129" gate="G$1" x="38.1" y="40.64" rot="R270"/>
 </instances>
 <busses>
@@
 </segment>
 <segment>
-<pinref part="R127" gate="G$1" pin="1"/>
 <pinref part="V305" gate="1" pin="GND"/>
-<wire x1="22.86" y1="40.64" x2="22.86" y2="43.18" width="0.1524" layer="91"/>
+<wire x1="22.86" y1="38.1" x2="22.86" y2="43.18" width="0.1524" layer="91"/>
+<pinref part="C1" gate="G$1" pin="-"/>
 </segment>
 <segment>
@@
 </segment>
 </net>
-<net name="N$489" class="0">
-<segment>
-<wire x1="38.1" y1="48.26" x2="38.1" y2="43.18" width="0.1524" layer="91"/>
+<net name="N$490" class="0">
+<segment>
 <wire x1="38.1" y1="48.26" x2="43.18" y2="48.26" width="0.1524" layer="91"/>
-<pinref part="R129" gate="G$1" pin="1"/>
 <pinref part="R130" gate="G$1" pin="2"/>
 <pinref part="TM4" gate="1" pin="S"/>
+<pinref part="R129" gate="G$1" pin="1"/>
+<wire x1="38.1" y1="45.72" x2="38.1" y2="48.26" width="0.1524" layer="91"/>
 <junction x="38.1" y="48.26"/>
-</segment>
-</net>
-<net name="N$490" class="0">
-<segment>
-<wire x1="38.1" y1="33.02" x2="38.1" y2="27.94" width="0.1524" layer="91"/>
-<pinref part="R129" gate="G$1" pin="2"/>
-<pinref part="IC1" gate="A" pin="-IN"/>
 </segment>
 </net>
@@
 </segment>
 </net>
-<net name="N$228" class="0">
-<segment>
-<pinref part="R127" gate="G$1" pin="2"/>
-<pinref part="TM4" gate="1" pin="A"/>
-</segment>
-</net>
 <net name="N$280" class="0">
 <segment>
@@
 </segment>
 </net>
+<net name="N$1" class="0">
+<segment>
+<pinref part="TM4" gate="1" pin="A"/>
+<pinref part="C1" gate="G$1" pin="+"/>
+<wire x1="30.48" y1="43.18" x2="33.02" y2="43.18" width="0.1524" layer="91"/>
+</segment>
+</net>
+<net name="N$2" class="0">
+<segment>
+<pinref part="R129" gate="G$1" pin="2"/>
+<pinref part="IC1" gate="A" pin="-IN"/>
+<wire x1="38.1" y1="35.56" x2="38.1" y2="27.94" width="0.1524" layer="91"/>
+</segment>
+</net>
